File: one-counter.sch (KiCad schematic (older format))
At the start: 9 parts

Commit message: associate symbols and add pullup to power on 7447
Parts:
- added R3: 150, symbol Device:R
- gave numbers to parts that had none: 9
Connections:
- wire segments 64 -> 66
Other:
- note removed: "Pin 16 has a 150 ohm pullup to 5V"
Changed lines of the file:
@@
 $EndDescr
 $Comp
-L Regulator_Linear:L7805 U?
+L Regulator_Linear:L7805 U1
 U 1 1 5B99A35E
 P 1850 6000
-F 0 "U?" H 1850 6242 50  0000 C CNN
+F 0 "U1" H 1850 6242 50  0000 C CNN
 F 1 "L7805" H 1850 6151 50  0000 C CNN
 F 2 "" H 1875 5850 50  0001 L CIN
@@
 $EndComp
 $Comp
-L Timer:LM555 U?
+L Timer:LM555 U2
 U 1 1 5B99A441
 P 3500 2400
-F 0 "U?" H 3500 2978 50  0000 C CNN
+F 0 "U2" H 3500 2978 50  0000 C CNN
 F 1 "LM555" H 3500 2887 50  0000 C CNN
 F 2 "" H 3500 2400 50  0001 C CNN
@@
 $EndComp
 $Comp
-L 74xx:74LS90 U?
+L 74xx:74LS90 U3
 U 1 1 5B99A4E4
 P 5850 2500
-F 0 "U?" H 5850 3278 50  0000 C CNN
+F 0 "U3" H 5850 3278 50  0000 C CNN
 F 1 "74LS90" H 5850 3187 50  0000 C CNN
 F 2 "" H 5850 2500 50  0001 C CNN
@@
 $EndComp
 $Comp
-L 74xx_IEEE:7447 U?
+L 74xx_IEEE:7447 U4
 U 1 1 5B99A664
 P 7300 2550
-F 0 "U?" H 7300 3166 50  0000 C CNN
+F 0 "U4" H 7300 3166 50  0000 C CNN
 F 1 "7447" H 7300 3075 50  0000 C CNN
 F 2 "" H 7300 2550 50  0001 C CNN
@@
 $EndComp
 $Comp
-L power:GND #PWR?
+L power:GND #PWR02
 U 1 1 5B99A8A7
 P 1850 6700
-F 0 "#PWR?" H 1850 6450 50  0001 C CNN
+F 0 "#PWR02" H 1850 6450 50  0001 C CNN
 F 1 "GND" H 1855 6527 50  0000 C CNN
 F 2 "" H 1850 6700 50  0001 C CNN
@@
 	1850 6300 1850 6700
 $Comp
-L power:+VDC #PWR?
+L power:+VDC #PWR01
 U 1 1 5B99A95B
 P 1400 5800
-F 0 "#PWR?" H 1400 5700 50  0001 C CNN
+F 0 "#PWR01" H 1400 5700 50  0001 C CNN
 F 1 "+VDC" H 1400 6075 50  0000 C CNN
 F 2 "" H 1400 5800 50  0001 C CNN
@@
 	1400 6000 1550 6000
 $Comp
-L power:+5V #PWR?
+L power:+5V #PWR04
 U 1 1 5B99A9A9
 P 2350 5750
-F 0 "#PWR?" H 2350 5600 50  0001 C CNN
+F 0 "#PWR04" H 2350 5600 50  0001 C CNN
 F 1 "+5V" H 2365 5923 50  0000 C CNN
 F 2 "" H 2350 5750 50  0001 C CNN
@@
 	2350 6000 2350 5750
 $Comp
-L power:+5V #PWR?
+L power:+5V #PWR06
 U 1 1 5B99A9EC
 P 3500 1550
-F 0 "#PWR?" H 3500 1400 50  0001 C CNN
+F 0 "#PWR06" H 3500 1400 50  0001 C CNN
 F 1 "+5V" H 3515 1723 50  0000 C CNN
 F 2 "" H 3500 1550 50  0001 C CNN
@@
 	3500 2000 3500 1750
 $Comp
-L power:+5V #PWR?
+L power:+5V #PWR08
 U 1 1 5B99AA47
 P 5850 1650
-F 0 "#PWR?" H 5850 1500 50  0001 C CNN
+F 0 "#PWR08" H 5850 1500 50  0001 C CNN
 F 1 "+5V" H 5865 1823 50  0000 C CNN
 F 2 "" H 5850 1650 50  0001 C CNN
@@
 	5850 1900 5850 1650
 $Comp
-L power:GND #PWR?
+L power:GND #PWR07
 U 1 1 5B99AAD3
 P 3500 3200
-F 0 "#PWR?" H 3500 2950 50  0001 C CNN
+F 0 "#PWR07" H 3500 2950 50  0001 C CNN
 F 1 "GND" H 3505 3027 50  0000 C CNN
 F 2 "" H 3500 3200 50  0001 C CNN
@@
 	3500 2800 3500 3200
 $Comp
-L power:GND #PWR?
+L power:GND #PWR09
 U 1 1 5B99AB15
 P 5850 3600
-F 0 "#PWR?" H 5850 3350 50  0001 C CNN
+F 0 "#PWR09" H 5850 3350 50  0001 C CNN
 F 1 "GND" H 5855 3427 50  0000 C CNN
 F 2 "" H 5850 3600 50  0001 C CNN
@@
 	6350 2400 6750 2400
 $Comp
-L Display_Character:MAN71A U?
+L Display_Character:MAN71A U5
 U 1 1 5B99DCBE
 P 8800 2650
-F 0 "U?" H 8800 3317 50  0000 C CNN
+F 0 "U5" H 8800 3317 50  0000 C CNN
 F 1 "MAN71A" H 8800 3226 50  0000 C CNN
 F 2 "Display_7Segment:MAN71A" H 8300 1950 50  0001 L CNN
@@
 	1    0    0    -1
 $EndComp
-Text Notes 7050 1850 0    50   ~ 0
-Pin 16 has a 150 ohm pullup to 5V
 Text Notes 8600 1850 0    50   ~ 0
 Using part 5082-7620 (package drawing E). Everything about this symbol is correct except DP (but I'm not using DP). Layout prob wrong.
@@
 NoConn ~ 8500 3050
 $Comp
-L power:+5V #PWR?
+L power:+5V #PWR010
 U 1 1 5B9A1426
 P 9250 2500
-F 0 "#PWR?" H 9250 2350 50  0001 C CNN
+F 0 "#PWR010" H 9250 2350 50  0001 C CNN
 F 1 "+5V" H 9265 2673 50  0000 C CNN
 F 2 "" H 9250 2500 50  0001 C CNN
@@
 	2800 2600 3000 2600
 $Comp
-L Device:R R?
+L Device:R R1
 U 1 1 5B9AE6CC
 P 4300 2000
-F 0 "R?" H 4370 2046 50  0000 L CNN
+F 0 "R1" H 4370 2046 50  0000 L CNN
 F 1 "1k" H 4370 1955 50  0000 L CNN
 F 2 "" V 4230 2000 50  0001 C CNN
@@
 $EndComp
 $Comp
-L Device:R R?
+L Device:R R2
 U 1 1 5B9AE762
 P 4300 2400
-F 0 "R?" H 4370 2446 50  0000 L CNN
+F 0 "R2" H 4370 2446 50  0000 L CNN
 F 1 "330k" H 4370 2355 50  0000 L CNN
 F 2 "" V 4230 2400 50  0001 C CNN
@@
 $EndComp
 $Comp
-L Device:C C?
+L Device:C C2
 U 1 1 5B9AE7E4
 P 2450 2650
-F 0 "C?" H 2565 2696 50  0000 L CNN
+F 0 "C2" H 2565 2696 50  0000 L CNN
 F 1 "0.01uF" H 2565 2605 50  0000 L CNN
 F 2 "" H 2488 2500 50  0001 C CNN
@@
 $EndComp
 $Comp
-L Device:CP C?
+L Device:CP C1
 U 1 1 5B9AE85A
 P 1900 2650
-F 0 "C?" H 2018 2696 50  0000 L CNN
+F 0 "C1" H 2018 2696 50  0000 L CNN
 F 1 "2.2uF" H 2018 2605 50  0000 L CNN
 F 2 "" H 1938 2500 50  0001 C CNN
@@
 $EndComp
 $Comp
-L power:GND #PWR?
+L power:GND #PWR05
 U 1 1 5B9AE8E0
 P 2450 3200
-F 0 "#PWR?" H 2450 2950 50  0001 C CNN
+F 0 "#PWR05" H 2450 2950 50  0001 C CNN
 F 1 "GND" H 2455 3027 50  0000 C CNN
 F 2 "" H 2450 3200 50  0001 C CNN
@@
 	2450 2800 2450 3200
 $Comp
-L power:GND #PWR?
+L power:GND #PWR03
 U 1 1 5B9AF078
 P 1900 3200
-F 0 "#PWR?" H 1900 2950 50  0001 C CNN
+F 0 "#PWR03" H 1900 2950 50  0001 C CNN
 F 1 "GND" H 1905 3027 50  0000 C CNN
 F 2 "" H 1900 3200 50  0001 C CNN
@@
 Wire Wire Line
 	4300 1650 4300 1850
+$Comp
+L Device:R R3
+U 1 1 5B9BEA7F
+P 7300 1650
+F 0 "R3" H 7370 1696 50  0000 L CNN
+F 1 "150" H 7370 1605 50  0000 L CNN
+F 2 "" V 7230 1650 50  0001 C CNN
+F 3 "~" H 7300 1650 50  0001 C CNN
+	1    7300 1650
+	1    0    0    -1
+$EndComp
+$Comp
+L power:+5V #PWR0101
+U 1 1 5B9BFF73
+P 7300 1250
+F 0 "#PWR0101" H 7300 1100 50  0001 C CNN
+F 1 "+5V" H 7315 1423 50  0000 C CNN
+F 2 "" H 7300 1250 50  0001 C CNN
+F 3 "" H 7300 1250 50  0001 C CNN
+	1    7300 1250
+	1    0    0    -1
+$EndComp
+Wire Wire Line
+	7300 1800 7300 2150
+Wire Wire Line
+	7300 1250 7300 1500
 $EndSCHEMATC

Commit message: add power flags
Connections:
- wire segments 66 -> 71
Changed lines of the file:
@@
 $EndComp
 Wire Wire Line
-	1850 6300 1850 6700
+	1850 6300 1850 6600
 $Comp
 L power:+VDC #PWR01
 U 1 1 5B99A95B
-P 1400 5800
-F 0 "#PWR01" H 1400 5700 50  0001 C CNN
-F 1 "+VDC" H 1400 6075 50  0000 C CNN
-F 2 "" H 1400 5800 50  0001 C CNN
-F 3 "" H 1400 5800 50  0001 C CNN
-	1    1400 5800
-	1    0    0    -1
-$EndComp
-Wire Wire Line
-	1400 5800 1400 6000
-Wire Wire Line
-	1400 6000 1550 6000
+P 1150 5800
+F 0 "#PWR01" H 1150 5700 50  0001 C CNN
+F 1 "+VDC" H 1150 6075 50  0000 C CNN
+F 2 "" H 1150 5800 50  0001 C CNN
+F 3 "" H 1150 5800 50  0001 C CNN
+	1    1150 5800
+	1    0    0    -1
+$EndComp
 $Comp
 L power:+5V #PWR04
 U 1 1 5B99A9A9
-P 2350 5750
-F 0 "#PWR04" H 2350 5600 50  0001 C CNN
-F 1 "+5V" H 2365 5923 50  0000 C CNN
-F 2 "" H 2350 5750 50  0001 C CNN
-F 3 "" H 2350 5750 50  0001 C CNN
-	1    2350 5750
-	1    0    0    -1
-$EndComp
-Wire Wire Line
-	2150 6000 2350 6000
-Wire Wire Line
-	2350 6000 2350 5750
+P 2600 5700
+F 0 "#PWR04" H 2600 5550 50  0001 C CNN
+F 1 "+5V" H 2615 5873 50  0000 C CNN
+F 2 "" H 2600 5700 50  0001 C CNN
+F 3 "" H 2600 5700 50  0001 C CNN
+	1    2600 5700
+	1    0    0    -1
+$EndComp
 $Comp
 L power:+5V #PWR06
@@
 Wire Wire Line
 	7300 1250 7300 1500
+$Comp
+L power:PWR_FLAG #FLG0101
+U 1 1 5B9C2C14
+P 2350 6000
+F 0 "#FLG0101" H 2350 6075 50  0001 C CNN
+F 1 "PWR_FLAG" H 2350 6174 50  0000 C CNN
+F 2 "" H 2350 6000 50  0001 C CNN
+F 3 "~" H 2350 6000 50  0001 C CNN
+	1    2350 6000
+	1    0    0    -1
+$EndComp
+$Comp
+L power:PWR_FLAG #FLG0102
+U 1 1 5B9C2C6E
+P 1400 6000
+F 0 "#FLG0102" H 1400 6075 50  0001 C CNN
+F 1 "PWR_FLAG" H 1400 6174 50  0000 C CNN
+F 2 "" H 1400 6000 50  0001 C CNN
+F 3 "~" H 1400 6000 50  0001 C CNN
+	1    1400 6000
+	1    0    0    -1
+$EndComp
+Wire Wire Line
+	2600 6000 2600 5700
+Wire Wire Line
+	2350 6000 2600 6000
+$Comp
+L power:PWR_FLAG #FLG0103
+U 1 1 5B9C6BEF
+P 2250 6550
+F 0 "#FLG0103" H 2250 6625 50  0001 C CNN
+F 1 "PWR_FLAG" H 2250 6724 50  0000 C CNN
+F 2 "" H 2250 6550 50  0001 C CNN
+F 3 "~" H 2250 6550 50  0001 C CNN
+	1    2250 6550
+	1    0    0    -1
+$EndComp
+Wire Wire Line
+	2250 6550 2250 6600
+Wire Wire Line
+	2250 6600 1850 6600
+Connection ~ 1850 6600
+Wire Wire Line
+	1850 6600 1850 6700
+Wire Wire Line
+	1400 6000 1550 6000
+Connection ~ 2350 6000
+Wire Wire Line
+	2150 6000 2350 6000
+Wire Wire Line
+	1150 5800 1150 6000
+Wire Wire Line
+	1150 6000 1400 6000
+Connection ~ 1400 6000
 $EndSCHEMATC

Commit message: applied physical footprints
Parts:
- C1: footprint (none) -> Capacitors_SMD:CP_Elec_4x5.8
- C2: footprint (none) -> Capacitors_THT:C_Disc_D3.0mm_W1.6mm_P2.50mm
- R1, R2, R3: footprint (none) -> Resistors_THT:R_Axial_DIN0204_L3.6mm_D1.6mm_P1.90mm_Vertical
- U1: footprint (none) -> digikey-footprints:TO-220-3
- U2: footprint (none) -> digikey-footprints:DIP-8_W7.62mm
- U3: footprint (none) -> Housings_DIP:DIP-14_W7.62mm
- U4: footprint (none) -> Housings_DIP:DIP-16_W7.62mm
Changed lines of the file:
@@
 F 0 "U1" H 1850 6242 50  0000 C CNN
 F 1 "L7805" H 1850 6151 50  0000 C CNN
-F 2 "" H 1875 5850 50  0001 L CIN
+F 2 "digikey-footprints:TO-220-3" H 1875 5850 50  0001 L CIN
 F 3 "http://www.st.com/content/ccc/resource/technical/document/datasheet/41/4f/b3/b0/12/d4/47/88/CD00000444.pdf/files/CD00000444.pdf/jcr:content/translations/en.CD00000444.pdf" H 1850 5950 50  0001 C CNN
 	1    1850 6000
@@
 F 0 "U2" H 3500 2978 50  0000 C CNN
 F 1 "LM555" H 3500 2887 50  0000 C CNN
-F 2 "" H 3500 2400 50  0001 C CNN
+F 2 "digikey-footprints:DIP-8_W7.62mm" H 3500 2400 50  0001 C CNN
 F 3 "http://www.ti.com/lit/ds/symlink/lm555.pdf" H 3500 2400 50  0001 C CNN
 	1    3500 2400
@@
 F 0 "U3" H 5850 3278 50  0000 C CNN
 F 1 "74LS90" H 5850 3187 50  0000 C CNN
-F 2 "" H 5850 2500 50  0001 C CNN
+F 2 "Housings_DIP:DIP-14_W7.62mm" H 5850 2500 50  0001 C CNN
 F 3 "http://www.ti.com/lit/gpn/sn74LS90" H 5850 2500 50  0001 C CNN
 	1    5850 2500
@@
 F 0 "U4" H 7300 3166 50  0000 C CNN
 F 1 "7447" H 7300 3075 50  0000 C CNN
-F 2 "" H 7300 2550 50  0001 C CNN
+F 2 "Housings_DIP:DIP-16_W7.62mm" H 7300 2550 50  0001 C CNN
 F 3 "" H 7300 2550 50  0001 C CNN
 	1    7300 2550
@@
 F 0 "R1" H 4370 2046 50  0000 L CNN
 F 1 "1k" H 4370 1955 50  0000 L CNN
-F 2 "" V 4230 2000 50  0001 C CNN
+F 2 "Resistors_THT:R_Axial_DIN0204_L3.6mm_D1.6mm_P1.90mm_Vertical" V 4230 2000 50  0001 C CNN
 F 3 "~" H 4300 2000 50  0001 C CNN
 	1    4300 2000
@@
 F 0 "R2" H 4370 2446 50  0000 L CNN
 F 1 "330k" H 4370 2355 50  0000 L CNN
-F 2 "" V 4230 2400 50  0001 C CNN
+F 2 "Resistors_THT:R_Axial_DIN0204_L3.6mm_D1.6mm_P1.90mm_Vertical" V 4230 2400 50  0001 C CNN
 F 3 "~" H 4300 2400 50  0001 C CNN
 	1    4300 2400
@@
 F 0 "C2" H 2565 2696 50  0000 L CNN
 F 1 "0.01uF" H 2565 2605 50  0000 L CNN
-F 2 "" H 2488 2500 50  0001 C CNN
+F 2 "Capacitors_THT:C_Disc_D3.0mm_W1.6mm_P2.50mm" H 2488 2500 50  0001 C CNN
 F 3 "~" H 2450 2650 50  0001 C CNN
 	1    2450 2650
@@
 F 0 "C1" H 2018 2696 50  0000 L CNN
 F 1 "2.2uF" H 2018 2605 50  0000 L CNN
-F 2 "" H 1938 2500 50  0001 C CNN
+F 2 "Capacitors_SMD:CP_Elec_4x5.8" H 1938 2500 50  0001 C CNN
 F 3 "~" H 1900 2650 50  0001 C CNN
 	1    1900 2650
@@
 F 0 "R3" H 7370 1696 50  0000 L CNN
 F 1 "150" H 7370 1605 50  0000 L CNN
-F 2 "" V 7230 1650 50  0001 C CNN
+F 2 "Resistors_THT:R_Axial_DIN0204_L3.6mm_D1.6mm_P1.90mm_Vertical" V 7230 1650 50  0001 C CNN
 F 3 "~" H 7300 1650 50  0001 C CNN
 	1    7300 1650

Commit message: update netlist
Parts:
- U5: footprint Display_7Segment:MAN71A -> digikey-footprints:LED_7Seg_VAOS-C402S9-BW_50
Changed lines of the file:
@@
 F 0 "U5" H 8800 3317 50  0000 C CNN
 F 1 "MAN71A" H 8800 3226 50  0000 C CNN
-F 2 "Display_7Segment:MAN71A" H 8300 1950 50  0001 L CNN
+F 2 "digikey-footprints:LED_7Seg_VAOS-C402S9-BW_50" H 8300 1950 50  0001 L CNN
 F 3 "https://www.digchip.com/datasheets/parts/datasheet/161/MAN3640A-pdf.php" H 8810 2990 50  0001 L CNN
 	1    8800 2650

Commit message: use new 555 in sch
Parts:
- removed U2: LM555, digikey-footprints:DIP-8_W7.62mm, symbol Timer:LM555
- added U?: 555-L, symbol one-counter:555-L
- added U?: 555-R, symbol one-counter:555-R
Connections:
- net labels added: 1Hz
- wire segments 71 -> 73
Other:
- note removed: "1Hz"
Changed lines of the file:
@@
-$EndComp
-$Comp
-L Timer:LM555 U2
-U 1 1 5B99A441
-P 3500 2400
-F 0 "U2" H 3500 2978 50  0000 C CNN
-F 1 "LM555" H 3500 2887 50  0000 C CNN
-F 2 "digikey-footprints:DIP-8_W7.62mm" H 3500 2400 50  0001 C CNN
-F 3 "http://www.ti.com/lit/ds/symlink/lm555.pdf" H 3500 2400 50  0001 C CNN
-	1    3500 2400
-	1    0    0    -1
 $EndComp
 $Comp
@@
 L power:+5V #PWR06
 U 1 1 5B99A9EC
-P 3500 1550
-F 0 "#PWR06" H 3500 1400 50  0001 C CNN
-F 1 "+5V" H 3515 1723 50  0000 C CNN
-F 2 "" H 3500 1550 50  0001 C CNN
-F 3 "" H 3500 1550 50  0001 C CNN
-	1    3500 1550
-	1    0    0    -1
-$EndComp
-Wire Wire Line
-	3500 2000 3500 1750
+P 3900 1600
+F 0 "#PWR06" H 3900 1450 50  0001 C CNN
+F 1 "+5V" H 3915 1773 50  0000 C CNN
+F 2 "" H 3900 1600 50  0001 C CNN
+F 3 "" H 3900 1600 50  0001 C CNN
+	1    3900 1600
+	1    0    0    -1
+$EndComp
 $Comp
 L power:+5V #PWR08
@@
 L power:GND #PWR07
 U 1 1 5B99AAD3
-P 3500 3200
-F 0 "#PWR07" H 3500 2950 50  0001 C CNN
-F 1 "GND" H 3505 3027 50  0000 C CNN
-F 2 "" H 3500 3200 50  0001 C CNN
-F 3 "" H 3500 3200 50  0001 C CNN
-	1    3500 3200
-	1    0    0    -1
-$EndComp
-Wire Wire Line
-	3500 2800 3500 3200
+P 2050 2150
+F 0 "#PWR07" H 2050 1900 50  0001 C CNN
+F 1 "GND" H 2055 1977 50  0000 C CNN
+F 2 "" H 2050 2150 50  0001 C CNN
+F 3 "" H 2050 2150 50  0001 C CNN
+	1    2050 2150
+	1    0    0    -1
+$EndComp
 $Comp
 L power:GND #PWR09
@@
 NoConn ~ 6750 2750
 NoConn ~ 6750 2850
-Text Notes 4000 2200 0    50   ~ 0
-1Hz
 Text Notes 1000 5400 0    50   ~ 0
 Didn't use capacitors before but probably should
@@
 Text Notes 9300 3000 0    50   ~ 0
 Only need to connect one of these anodes to +5V
-Wire Wire Line
-	4000 2200 5350 2200
-Wire Wire Line
-	2800 2600 3000 2600
 $Comp
 L Device:R R1
 U 1 1 5B9AE6CC
-P 4300 2000
-F 0 "R1" H 4370 2046 50  0000 L CNN
-F 1 "1k" H 4370 1955 50  0000 L CNN
-F 2 "Resistors_THT:R_Axial_DIN0204_L3.6mm_D1.6mm_P1.90mm_Vertical" V 4230 2000 50  0001 C CNN
-F 3 "~" H 4300 2000 50  0001 C CNN
-	1    4300 2000
+P 4350 2000
+F 0 "R1" H 4420 2046 50  0000 L CNN
+F 1 "1k" H 4420 1955 50  0000 L CNN
+F 2 "Resistors_THT:R_Axial_DIN0204_L3.6mm_D1.6mm_P1.90mm_Vertical" V 4280 2000 50  0001 C CNN
+F 3 "~" H 4350 2000 50  0001 C CNN
+	1    4350 2000
 	1    0    0    -1
 $EndComp
@@
 L Device:R R2
 U 1 1 5B9AE762
-P 4300 2400
-F 0 "R2" H 4370 2446 50  0000 L CNN
-F 1 "330k" H 4370 2355 50  0000 L CNN
-F 2 "Resistors_THT:R_Axial_DIN0204_L3.6mm_D1.6mm_P1.90mm_Vertical" V 4230 2400 50  0001 C CNN
-F 3 "~" H 4300 2400 50  0001 C CNN
-	1    4300 2400
+P 4350 2400
+F 0 "R2" H 4420 2446 50  0000 L CNN
+F 1 "330k" H 4420 2355 50  0000 L CNN
+F 2 "Resistors_THT:R_Axial_DIN0204_L3.6mm_D1.6mm_P1.90mm_Vertical" V 4280 2400 50  0001 C CNN
+F 3 "~" H 4350 2400 50  0001 C CNN
+	1    4350 2400
 	1    0    0    -1
 $EndComp
@@
 L Device:C C2
 U 1 1 5B9AE7E4
-P 2450 2650
-F 0 "C2" H 2565 2696 50  0000 L CNN
-F 1 "0.01uF" H 2565 2605 50  0000 L CNN
-F 2 "Capacitors_THT:C_Disc_D3.0mm_W1.6mm_P2.50mm" H 2488 2500 50  0001 C CNN
-F 3 "~" H 2450 2650 50  0001 C CNN
-	1    2450 2650
+P 3900 2900
+F 0 "C2" H 4015 2946 50  0000 L CNN
+F 1 "0.01uF" H 4015 2855 50  0000 L CNN
+F 2 "Capacitors_THT:C_Disc_D3.0mm_W1.6mm_P2.50mm" H 3938 2750 50  0001 C CNN
+F 3 "~" H 3900 2900 50  0001 C CNN
+	1    3900 2900
 	1    0    0    -1
 $EndComp
@@
 L Device:CP C1
 U 1 1 5B9AE85A
-P 1900 2650
-F 0 "C1" H 2018 2696 50  0000 L CNN
-F 1 "2.2uF" H 2018 2605 50  0000 L CNN
-F 2 "Capacitors_SMD:CP_Elec_4x5.8" H 1938 2500 50  0001 C CNN
-F 3 "~" H 1900 2650 50  0001 C CNN
-	1    1900 2650
+P 4350 2950
+F 0 "C1" H 4468 2996 50  0000 L CNN
+F 1 "2.2uF" H 4468 2905 50  0000 L CNN
+F 2 "Capacitors_SMD:CP_Elec_4x5.8" H 4388 2800 50  0001 C CNN
+F 3 "~" H 4350 2950 50  0001 C CNN
+	1    4350 2950
 	1    0    0    -1
 $EndComp
@@
 L power:GND #PWR05
 U 1 1 5B9AE8E0
-P 2450 3200
-F 0 "#PWR05" H 2450 2950 50  0001 C CNN
-F 1 "GND" H 2455 3027 50  0000 C CNN
-F 2 "" H 2450 3200 50  0001 C CNN
-F 3 "" H 2450 3200 50  0001 C CNN
-	1    2450 3200
-	1    0    0    -1
-$EndComp
-Wire Wire Line
-	2450 2800 2450 3200
+P 3900 3300
+F 0 "#PWR05" H 3900 3050 50  0001 C CNN
+F 1 "GND" H 3905 3127 50  0000 C CNN
+F 2 "" H 3900 3300 50  0001 C CNN
+F 3 "" H 3900 3300 50  0001 C CNN
+	1    3900 3300
+	1    0    0    -1
+$EndComp
+Wire Wire Line
+	3900 3050 3900 3300
 $Comp
 L power:GND #PWR03
 U 1 1 5B9AF078
-P 1900 3200
-F 0 "#PWR03" H 1900 2950 50  0001 C CNN
-F 1 "GND" H 1905 3027 50  0000 C CNN
-F 2 "" H 1900 3200 50  0001 C CNN
-F 3 "" H 1900 3200 50  0001 C CNN
-	1    1900 3200
-	1    0    0    -1
-$EndComp
-Wire Wire Line
-	1900 2800 1900 3200
-Wire Wire Line
-	2450 2500 2450 2400
-Wire Wire Line
-	2450 2400 3000 2400
-Wire Wire Line
-	3000 2200 2900 2200
-Wire Wire Line
-	1900 2200 1900 2500
-Wire Wire Line
-	4000 2600 4100 2600
-Wire Wire Line
-	4300 2600 4300 2550
-Wire Wire Line
-	4300 2250 4300 2150
-Wire Wire Line
-	4000 2400 4100 2400
-Wire Wire Line
-	4100 2400 4100 2250
-Wire Wire Line
-	4100 2250 4300 2250
-Connection ~ 4300 2250
-Wire Wire Line
-	4300 1650 3500 1650
-Connection ~ 3500 1650
-Wire Wire Line
-	3500 1650 3500 1550
-Wire Wire Line
-	2900 2200 2900 2850
-Wire Wire Line
-	2900 2850 4100 2850
-Wire Wire Line
-	4100 2850 4100 2600
-Connection ~ 2900 2200
-Wire Wire Line
-	2900 2200 1900 2200
-Connection ~ 4100 2600
-Wire Wire Line
-	4100 2600 4300 2600
-Wire Wire Line
-	3500 1750 2800 1750
-Connection ~ 3500 1750
-Wire Wire Line
-	3500 1750 3500 1650
-Wire Wire Line
-	2800 1750 2800 2600
-Wire Wire Line
-	4300 1650 4300 1850
+P 4350 3200
+F 0 "#PWR03" H 4350 2950 50  0001 C CNN
+F 1 "GND" H 4355 3027 50  0000 C CNN
+F 2 "" H 4350 3200 50  0001 C CNN
+F 3 "" H 4350 3200 50  0001 C CNN
+	1    4350 3200
+	1    0    0    -1
+$EndComp
+Wire Wire Line
+	4350 3100 4350 3200
+Wire Wire Line
+	2300 2200 2300 2600
+Wire Wire Line
+	4350 2600 4350 2550
+Wire Wire Line
+	4350 2250 4350 2200
 $Comp
 L Device:R R3
@@
 	1150 6000 1400 6000
 Connection ~ 1400 6000
+$Comp
+L one-counter:555-L U?
+U 1 1 5B9AC94F
+P 3250 2050
+F 0 "U?" H 3050 2100 50  0000 L CNN
+F 1 "555-L" H 2950 1600 50  0000 L CNN
+F 2 "" H 3150 2050 50  0001 C CNN
+F 3 "" H 3150 2050 50  0001 C CNN
+	1    3250 2050
+	1    0    0    -1
+$EndComp
+$Comp
+L one-counter:555-R U?
+U 1 1 5B9AC9D3
+P 3250 2050
+F 0 "U?" H 3500 2100 50  0000 C CNN
+F 1 "555-R" H 3450 1600 50  0000 C CNN
+F 2 "" H 3250 2050 50  0001 C CNN
+F 3 "" H 3250 2050 50  0001 C CNN
+	1    3250 2050
+	1    0    0    -1
+$EndComp
+Connection ~ 4350 2200
+Wire Wire Line
+	4350 2200 4350 2150
+Wire Wire Line
+	4350 1800 4350 1850
+Wire Wire Line
+	2700 2400 2600 2400
+Wire Wire Line
+	2600 2400 2600 1900
+Wire Wire Line
+	2600 1900 3900 1900
+Connection ~ 3900 1900
+Wire Wire Line
+	3900 1900 3900 2100
+Wire Wire Line
+	3900 2300 4050 2300
+Wire Wire Line
+	4050 2300 4050 2600
+Wire Wire Line
+	3900 2400 3900 2750
+Wire Wire Line
+	2700 2200 2300 2200
+Wire Wire Line
+	4050 2600 2300 2600
+Wire Wire Line
+	4350 2600 4350 2800
+Connection ~ 4350 2600
+Wire Wire Line
+	3900 1600 3900 1800
+Wire Wire Line
+	3900 1800 4350 1800
+Connection ~ 3900 1800
+Wire Wire Line
+	3900 1800 3900 1900
+Wire Wire Line
+	3900 2200 4350 2200
+Wire Wire Line
+	4050 2600 4350 2600
+Connection ~ 4050 2600
+Wire Wire Line
+	2700 2300 2450 2300
+Wire Wire Line
+	2450 2300 2450 1750
+Wire Wire Line
+	2450 1750 4900 1750
+Wire Wire Line
+	4900 1750 4900 2200
+Wire Wire Line
+	4900 2200 4950 2200
+Wire Wire Line
+	2050 2100 2050 2150
+Wire Wire Line
+	2050 2100 2700 2100
+Text Label 2500 1750 0    50   ~ 0
+1Hz
 $EndSCHEMATC

Commit message: redo schematic with custom parts
Parts:
- removed U3: 74LS90, Housings_DIP:DIP-14_W7.62mm, symbol 74xx:74LS90
- removed U4: 7447, Housings_DIP:DIP-16_W7.62mm, symbol 74xx_IEEE:7447
- removed U5: MAN71A, digikey-footprints:LED_7Seg_VAOS-C402S9-BW_50, symbol Display_Character:MAN71A
- added U?: 74LS90-L, symbol one-counter:74LS90-L
- added U?: 74LS90-R, symbol one-counter:74LS90-R
- added U?: 7447-L, symbol one-counter:7447-L
- added U?: 7447-R, symbol one-counter:7447-R
- added U?: 5082-7650-L, symbol one-counter:5082-7650-L
- added U?: 5082-7650-R, symbol one-counter:5082-7650-R
Connections:
- wire segments 73 -> 106
- no-connect marks 4 -> 8
Other:
- note removed: "Using part 5082-7620 (package drawing E). Everything about this symbol is correct except DP (but I'm not using DP). Layout prob wrong."

Commit message: annotate symbols
Parts:
- gave numbers to parts that had none: 8
- renumbered C2 to C1, C1 to C2

Commit message: assign 2.54mm headers to all parts
Parts:
- U2, U3: footprint (none) -> Pin_Headers:Pin_Header_Straight_1x04_Pitch2.54mm
- U4, U5, U8, U9: footprint (none) -> Pin_Headers:Pin_Header_Straight_1x07_Pitch2.54mm
- U6, U7: footprint (none) -> Pin_Headers:Pin_Header_Straight_1x08_Pitch2.54mm
Changed lines of the file:
@@
 F 0 "U2" H 3600 2050 50  0000 L CNN
 F 1 "555-L" H 3500 1550 50  0000 L CNN
-F 2 "" H 3700 2000 50  0001 C CNN
+F 2 "Pin_Headers:Pin_Header_Straight_1x04_Pitch2.54mm" H 3700 2000 50  0001 C CNN
 F 3 "" H 3700 2000 50  0001 C CNN
 	1    3800 2000
@@
 F 0 "U3" H 4050 2050 50  0000 C CNN
 F 1 "555-R" H 4000 1550 50  0000 C CNN
-F 2 "" H 3800 2000 50  0001 C CNN
+F 2 "Pin_Headers:Pin_Header_Straight_1x04_Pitch2.54mm" H 3800 2000 50  0001 C CNN
 F 3 "" H 3800 2000 50  0001 C CNN
 	1    3800 2000
@@
 F 0 "U4" H 6150 1950 50  0000 L CNN
 F 1 "74LS90-L" H 5900 1150 50  0000 L CNN
-F 2 "" H 6250 1900 50  0001 C CNN
+F 2 "Pin_Headers:Pin_Header_Straight_1x07_Pitch2.54mm" H 6250 1900 50  0001 C CNN
 F 3 "" H 6250 1900 50  0001 C CNN
 	1    6300 1900
@@
 F 0 "U5" H 6400 1950 50  0000 C CNN
 F 1 "74LS90-R" H 6500 1150 50  0000 C CNN
-F 2 "" H 6250 1900 50  0001 C CNN
+F 2 "Pin_Headers:Pin_Header_Straight_1x07_Pitch2.54mm" H 6250 1900 50  0001 C CNN
 F 3 "" H 6250 1900 50  0001 C CNN
 	1    6300 1900
@@
 F 0 "U6" H 7500 1950 50  0000 L CNN
 F 1 "7447-L" H 7400 1050 50  0000 L CNN
-F 2 "" H 7700 1900 50  0001 C CNN
+F 2 "Pin_Headers:Pin_Header_Straight_1x08_Pitch2.54mm" H 7700 1900 50  0001 C CNN
 F 3 "" H 7700 1900 50  0001 C CNN
 	1    7700 1900
@@
 F 0 "U7" H 7800 1950 50  0000 C CNN
 F 1 "7447-R" H 7850 1050 50  0000 C CNN
-F 2 "" H 7700 1900 50  0001 C CNN
+F 2 "Pin_Headers:Pin_Header_Straight_1x08_Pitch2.54mm" H 7700 1900 50  0001 C CNN
 F 3 "" H 7700 1900 50  0001 C CNN
 	1    7700 1900
@@
 F 0 "U8" H 9100 2050 50  0000 L CNN
 F 1 "5082-7650-L" H 8750 1250 50  0000 L CNN
-F 2 "" H 9300 2000 50  0001 C CNN
+F 2 "Pin_Headers:Pin_Header_Straight_1x07_Pitch2.54mm" H 9300 2000 50  0001 C CNN
 F 3 "" H 9300 2000 50  0001 C CNN
 	1    9300 2000
@@
 F 0 "U9" H 9450 2050 50  0000 C CNN
 F 1 "5082-7650-R" H 9600 1250 50  0000 C CNN
-F 2 "" H 9300 2000 50  0001 C CNN
+F 2 "Pin_Headers:Pin_Header_Straight_1x07_Pitch2.54mm" H 9300 2000 50  0001 C CNN
 F 3 "" H 9300 2000 50  0001 C CNN
 	1    9300 2000
