File: one-counter.sch (KiCad schematic (older format))
At the start: 14 parts, among them U1 L7805, U2 555-L, U3 555-R, U4 74LS90-L, U5 74LS90-R, U6 7447-L, U7 7447-R, U8 5082-7650-L, U9 5082-7650-R

Commit message: Add right side parts to layout
Parts:
- U3: footprint Pin_Headers:Pin_Header_Straight_1x04_Pitch2.54mm -> one-counter:Pin_Header_Straight_1x04_Pitch2.54mm_Right
- U5, U9: footprint Pin_Headers:Pin_Header_Straight_1x07_Pitch2.54mm -> one-counter:Pin_Header_Straight_1x07_Pitch2.54mm_Right
- U7: footprint Pin_Headers:Pin_Header_Straight_1x08_Pitch2.54mm -> one-counter:Pin_Header_Straight_1x08_Pitch2.54mm_Right
Changed lines of the file:
@@
 F 0 "U3" H 4050 2050 50  0000 C CNN
 F 1 "555-R" H 4000 1550 50  0000 C CNN
-F 2 "Pin_Headers:Pin_Header_Straight_1x04_Pitch2.54mm" H 3800 2000 50  0001 C CNN
+F 2 "one-counter:Pin_Header_Straight_1x04_Pitch2.54mm_Right" H 3800 2000 50  0001 C CNN
 F 3 "" H 3800 2000 50  0001 C CNN
 	1    3800 2000
@@
 F 0 "U5" H 6400 1950 50  0000 C CNN
 F 1 "74LS90-R" H 6500 1150 50  0000 C CNN
-F 2 "Pin_Headers:Pin_Header_Straight_1x07_Pitch2.54mm" H 6250 1900 50  0001 C CNN
+F 2 "one-counter:Pin_Header_Straight_1x07_Pitch2.54mm_Right" H 6250 1900 50  0001 C CNN
 F 3 "" H 6250 1900 50  0001 C CNN
 	1    6300 1900
@@
 F 0 "U7" H 7800 1950 50  0000 C CNN
 F 1 "7447-R" H 7850 1050 50  0000 C CNN
-F 2 "Pin_Headers:Pin_Header_Straight_1x08_Pitch2.54mm" H 7700 1900 50  0001 C CNN
+F 2 "one-counter:Pin_Header_Straight_1x08_Pitch2.54mm_Right" H 7700 1900 50  0001 C CNN
 F 3 "" H 7700 1900 50  0001 C CNN
 	1    7700 1900
@@
 F 0 "U9" H 9450 2050 50  0000 C CNN
 F 1 "5082-7650-R" H 9600 1250 50  0000 C CNN
-F 2 "Pin_Headers:Pin_Header_Straight_1x07_Pitch2.54mm" H 9300 2000 50  0001 C CNN
+F 2 "one-counter:Pin_Header_Straight_1x07_Pitch2.54mm_Right" H 9300 2000 50  0001 C CNN
 F 3 "" H 9300 2000 50  0001 C CNN
 	1    9300 2000

Commit message: routing is possible
Parts:
- added J1: Conn_01x08-L, Pin_Headers:Pin_Header_Straight_1x08_Pitch2.54mm, symbol Connector:Conn_01x08_Male
- added J2: Conn_01x08-R, Pin_Headers:Pin_Header_Straight_1x08_Pitch2.54mm, symbol Connector:Conn_01x08_Female
Connections:
- net labels added: U2-2, U3-6, U4-1, U5-12, U7-13, U7-15, U7-9, U8-1, U8-2, U8-7
- wire segments 106 -> 100

Commit message: don't need resistor
Parts:
- removed R3: 150, Resistors_THT:R_Axial_DIN0204_L3.6mm_D1.6mm_P1.90mm_Vertical, symbol Device:R
Connections:
- wire segments 100 -> 99
Changed lines of the file:
@@
 	1    0    0    -1
 $EndComp
-Wire Wire Line
-	8250 2600 8250 2850
 $Comp
 L power:PWR_FLAG #FLG03
@@
 $EndComp
 $Comp
-L Device:R R3
-U 1 1 5B9BEA7F
-P 8250 3000
-F 0 "R3" H 8320 3046 50  0000 L CNN
-F 1 "150" H 8320 2955 50  0000 L CNN
-F 2 "Resistors_THT:R_Axial_DIN0204_L3.6mm_D1.6mm_P1.90mm_Vertical" V 8180 3000 50  0001 C CNN
-F 3 "~" H 8250 3000 50  0001 C CNN
-	1    8250 3000
-	1    0    0    -1
-$EndComp
-$Comp
 L one-counter:7447-L U6
 U 1 1 5B9D034E
@@
 Wire Wire Line
 	8200 3350 8250 3350
-Wire Wire Line
-	8250 3350 8250 3150
 $Comp
 L one-counter:5082-7650-L U8
@@
 Text GLabel 4400 2150 2    50   Input ~ 0
 U8-2
+Wire Wire Line
+	8250 2600 8250 3350
 $EndSCHEMATC

Commit message: Run ERC/DRC and remove one anode connection
Connections:
- wire segments 99 -> 94
- no-connect marks 8 -> 9
Other:
- note removed: "Only need to connect one of these anodes to +5V"
Changed lines of the file:
@@
 L power:+5V #PWR016
 U 1 1 5B9A1426
-P 10950 2900
-F 0 "#PWR016" H 10950 2750 50  0001 C CNN
-F 1 "+5V" H 10965 3073 50  0000 C CNN
-F 2 "" H 10950 2900 50  0001 C CNN
-F 3 "" H 10950 2900 50  0001 C CNN
-	1    10950 2900
-	1    0    0    -1
-$EndComp
-Wire Wire Line
-	10950 2900 10950 3100
-Text Notes 8900 3050 0    50   ~ 0
-Only need to connect one of these anodes to +5V
+P 10250 3100
+F 0 "#PWR016" H 10250 2950 50  0001 C CNN
+F 1 "+5V" H 10265 3273 50  0000 C CNN
+F 2 "" H 10250 3100 50  0001 C CNN
+F 3 "" H 10250 3100 50  0001 C CNN
+	1    10250 3100
+	1    0    0    -1
+$EndComp
 $Comp
 L Device:R R1
@@
 L power:+5V #PWR015
 U 1 1 5B9BFF73
-P 8250 2600
-F 0 "#PWR015" H 8250 2450 50  0001 C CNN
-F 1 "+5V" H 8265 2773 50  0000 C CNN
-F 2 "" H 8250 2600 50  0001 C CNN
-F 3 "" H 8250 2600 50  0001 C CNN
-	1    8250 2600
-	1    0    0    -1
-$EndComp
-$Comp
-L power:PWR_FLAG #FLG03
-U 1 1 5B9C2C14
-P 2200 3450
-F 0 "#FLG03" H 2200 3525 50  0001 C CNN
-F 1 "PWR_FLAG" H 2200 3624 50  0000 C CNN
-F 2 "" H 2200 3450 50  0001 C CNN
-F 3 "~" H 2200 3450 50  0001 C CNN
-	1    2200 3450
+P 8250 3100
+F 0 "#PWR015" H 8250 2950 50  0001 C CNN
+F 1 "+5V" H 8265 3273 50  0000 C CNN
+F 2 "" H 8250 3100 50  0001 C CNN
+F 3 "" H 8250 3100 50  0001 C CNN
+	1    8250 3100
 	1    0    0    -1
 $EndComp
@@
 Wire Wire Line
 	2450 3450 2450 3150
-Wire Wire Line
-	2200 3450 2450 3450
 $Comp
 L power:PWR_FLAG #FLG02
@@
 Wire Wire Line
 	1250 3450 1400 3450
-Connection ~ 2200 3450
-Wire Wire Line
-	2000 3450 2200 3450
 Wire Wire Line
 	1000 3250 1000 3450
@@
 NoConn ~ 9900 3950
 Wire Wire Line
-	9900 3450 10950 3450
-Wire Wire Line
-	8900 3650 8850 3650
-Wire Wire Line
-	8850 3650 8850 3100
-Wire Wire Line
-	8850 3100 10950 3100
-Connection ~ 10950 3100
-Wire Wire Line
-	10950 3100 10950 3450
+	9900 3450 10250 3450
 $Comp
 L Connector:Conn_01x08_Male J1
@@
 U8-2
 Wire Wire Line
-	8250 2600 8250 3350
+	8250 3100 8250 3350
+Wire Wire Line
+	10250 3100 10250 3450
+NoConn ~ 8900 3650
+Wire Wire Line
+	2000 3450 2450 3450
 $EndSCHEMATC

Commit message: Change from 8 to 7 pin header
Parts:
- C1: footprint Capacitors_THT:C_Disc_D3.0mm_W1.6mm_P2.50mm -> Capacitor_THT:C_Disc_D7.5mm_W5.0mm_P5.00mm
- C2: footprint Capacitors_SMD:CP_Elec_4x5.8 -> Capacitor_THT:CP_Radial_D4.0mm_P1.50mm
- J1: value Conn_01x08-L -> Conn_01x07-L; footprint Pin_Headers:Pin_Header_Straight_1x08_Pitch2.54mm -> Connector_PinHeader_2.54mm:PinHeader_1x07_P2.54mm_Vertical; symbol Connector:Conn_01x08_Male -> Connector:Conn_01x07_Male
- J2: value Conn_01x08-R -> Conn_01x07-R; footprint Pin_Headers:Pin_Header_Straight_1x08_Pitch2.54mm -> Connector_PinHeader_2.54mm:PinHeader_1x07_P2.54mm_Vertical; symbol Connector:Conn_01x08_Female -> Connector:Conn_01x07_Female
Changed lines of the file:
@@
 F 0 "C1" H 4665 4296 50  0000 L CNN
 F 1 "0.01uF" H 4665 4205 50  0000 L CNN
-F 2 "Capacitors_THT:C_Disc_D3.0mm_W1.6mm_P2.50mm" H 4588 4100 50  0001 C CNN
+F 2 "Capacitor_THT:C_Disc_D7.5mm_W5.0mm_P5.00mm" H 4588 4100 50  0001 C CNN
 F 3 "~" H 4550 4250 50  0001 C CNN
 	1    4550 4250
@@
 F 0 "C2" H 5118 4346 50  0000 L CNN
 F 1 "2.2uF" H 5118 4255 50  0000 L CNN
-F 2 "Capacitors_SMD:CP_Elec_4x5.8" H 5038 4150 50  0001 C CNN
+F 2 "Capacitor_THT:CP_Radial_D4.0mm_P1.50mm" H 5038 4150 50  0001 C CNN
 F 3 "~" H 5000 4300 50  0001 C CNN
 	1    5000 4300
@@
 	9900 3450 10250 3450
 $Comp
-L Connector:Conn_01x08_Male J1
+L Connector:Conn_01x07_Male J1
 U 1 1 5BA28C02
 P 4200 1850
 F 0 "J1" H 4300 2300 50  0000 C CNN
-F 1 "Conn_01x08-L" H 4500 1350 50  0000 C CNN
-F 2 "Pin_Headers:Pin_Header_Straight_1x08_Pitch2.54mm" H 4200 1850 50  0001 C CNN
+F 1 "Conn_01x07-L" H 4500 1450 50  0000 C CNN
+F 2 "Connector_PinHeader_2.54mm:PinHeader_1x07_P2.54mm_Vertical" H 4200 1850 50  0001 C CNN
 F 3 "~" H 4200 1850 50  0001 C CNN
 	1    4200 1850
@@
 $EndComp
 $Comp
-L Connector:Conn_01x08_Female J2
+L Connector:Conn_01x07_Female J2
 U 1 1 5BA28D1D
 P 4200 1850
 F 0 "J2" H 4000 2300 50  0000 L CNN
-F 1 "Conn_01x08-R" H 3600 1350 50  0000 L CNN
-F 2 "Pin_Headers:Pin_Header_Straight_1x08_Pitch2.54mm" H 4200 1850 50  0001 C CNN
+F 1 "Conn_01x07-R" H 3600 1450 50  0000 L CNN
+F 2 "Connector_PinHeader_2.54mm:PinHeader_1x07_P2.54mm_Vertical" H 4200 1850 50  0001 C CNN
 F 3 "~" H 4200 1850 50  0001 C CNN
 	1    4200 1850

Commit message: changed resistor size
Parts:
- R1, R2: footprint Resistors_THT:R_Axial_DIN0204_L3.6mm_D1.6mm_P1.90mm_Vertical -> Resistor_THT:R_Axial_DIN0204_L3.6mm_D1.6mm_P2.54mm_Vertical
Changed lines of the file:
@@
 F 0 "R1" H 5070 3396 50  0000 L CNN
 F 1 "1k" H 5070 3305 50  0000 L CNN
-F 2 "Resistors_THT:R_Axial_DIN0204_L3.6mm_D1.6mm_P1.90mm_Vertical" V 4930 3350 50  0001 C CNN
+F 2 "Resistor_THT:R_Axial_DIN0204_L3.6mm_D1.6mm_P2.54mm_Vertical" V 4930 3350 50  0001 C CNN
 F 3 "~" H 5000 3350 50  0001 C CNN
 	1    5000 3350
@@
 F 0 "R2" H 5070 3796 50  0000 L CNN
 F 1 "330k" H 5070 3705 50  0000 L CNN
-F 2 "Resistors_THT:R_Axial_DIN0204_L3.6mm_D1.6mm_P1.90mm_Vertical" V 4930 3750 50  0001 C CNN
+F 2 "Resistor_THT:R_Axial_DIN0204_L3.6mm_D1.6mm_P2.54mm_Vertical" V 4930 3750 50  0001 C CNN
 F 3 "~" H 5000 3750 50  0001 C CNN
 	1    5000 3750

Commit message: move all components into place
Parts:
- C1: footprint Capacitor_THT:C_Disc_D7.5mm_W5.0mm_P5.00mm -> Capacitor_THT:C_Disc_D5.0mm_W2.5mm_P5.00mm
Changed lines of the file:
@@
 F 0 "C1" H 4665 4296 50  0000 L CNN
 F 1 "0.01uF" H 4665 4205 50  0000 L CNN
-F 2 "Capacitor_THT:C_Disc_D7.5mm_W5.0mm_P5.00mm" H 4588 4100 50  0001 C CNN
+F 2 "Capacitor_THT:C_Disc_D5.0mm_W2.5mm_P5.00mm" H 4588 4100 50  0001 C CNN
 F 3 "~" H 4550 4250 50  0001 C CNN
 	1    4550 4250
